File: sensorstrip.kicad_pcb (KiCad board)
At the start: 2 copper layers, 150 x 12 mm, 18 parts, among them J1 USB_C_Receptacle_PowerOnly, SW1 SW_DPDT_x2

Commit message: Update to v3
Parts:
- removed D1, D10, D5, D6, D7, D8, D9: LED, sensorstrip:LED_THT-1.27mm-OrthogonalSMDMount
- removed the R2 at (135.6, 52.2)
- removed the R3 at (215.4, 52.2)
- removed R4: 120R, Resistor_SMD:R_0603_1608Metric_Pad0.98x0.95mm_HandSolder
- added J2: Conn_01x02, Connector_JST:JST_GH_SM02B-GHS-TB_1x02-1MP_P1.25mm_Horizontal, F.Cu at (140.6, 53.8)
- added JP1: SolderJumper_2_Open, Jumper:SolderJumper-2_P1.3mm_Open_Pad1.0x1.5mm, F.Cu at (112.0, 56.1)
- moved J1 51.1 mm to (153.9, 57.4)
- moved R3 43.2 mm to (152.2, 60.1), turned to 0 degrees
- moved R2 36.6 mm to (155.8, 60.1), turned to 180 degrees
- moved SW1 33.1 mm to (113.2, 56.1)
- moved R1 22.3 mm to (133.8, 52.6), turned to 0 degrees
- moved D2 12.1 mm to (121.1, 58.0)
- moved D3 10.1 mm to (127.1, 58.0)
- moved D4 8.10 mm to (133.1, 58.0)
- renumbered R5 to R2, R6 to R3
Connections:
- D2 pad 2: /LEDs-R-Inner -> /LEDs
- D3 pad 2: /LEDs-R-Inner -> /LEDs
- D4 pad 2: /LEDs-R-Inner -> /LEDs
- R1 pad 1: +5V -> /LEDs
- R1 pad 2: /LEDs-R-Inner -> Power_postSwitch
- SW1 pad 1: +5V -> Power_postSwitch
- SW1 pad 4: +5V -> Power_postSwitch
Routing:
- net /LEDs-L-Outer: track 45.3 -> 0.00 mm
- net /LEDs-R-Outer: track 44.9 -> 0.00 mm
- net /LEDs-L-Inner: track 33.8 -> 0.00 mm
- net /LEDs-R-Inner: track 33.7 -> 0.00 mm
- net /LEDs: track 0.00 -> 26.8 mm
- net +5V: track 23.1 -> 0.00 mm, vias 5 -> 0
- net /VBUS: track 77.2 -> 58.6 mm
- net Power_postSwitch: track 0.00 -> 12.7 mm, vias 0 -> 3
- net /CC1: track 15.2 -> 2.95 mm
- net /CC2: track 10.1 -> 2.87 mm
- net GND: vias 11 -> 4
- added copper zone on F.Cu, net /VBUS
- added copper zone on B.Cu, net Power_postSwitch
- removed copper zone on B.Cu, net +5V
Other:
- board size 150 x 12 mm -> 55 x 12 mm

Commit message: Minor tweaks
Parts:
- renumbered D2 to D1, D3 to D2, D4 to D3
Connections:
- J2 pad MP: (no net) -> GND
Changed lines of the file:
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@@
     (property "Sheetname" "")
     (attr smd)
-    (fp_text reference "D3" (at -2.8 1.75 90 unlocked) (layer "F.SilkS")
+    (fp_text reference "D2" (at -2.8 1.75 90 unlocked) (layer "F.SilkS")
       (effects (font (size 1 1) (thickness 0.15)))
     )
@@
     (property "Sheetname" "")
     (attr smd)
-    (fp_text reference "D2" (at -2.8 1.85 90 unlocked) (layer "F.SilkS")
+    (fp_text reference "D1" (at -2.8 1.85 90 unlocked) (layer "F.SilkS")
       (effects (font (size 1 1) (thickness 0.15)))
     )
@@
     (pad "2" smd roundrect (at 0.625 -1.85 180) (size 0.6 1.7) (layers "F.Cu" "F.Paste" "F.Mask") (roundrect_rratio 0.25)
       (net 1 "GND") (pinfunction "Pin_2") (pintype "passive"))
-    (pad "MP" smd roundrect (at 2.475 1.35 180) (size 1 2.7) (layers "F.Cu" "F.Paste" "F.Mask") (roundrect_rratio 0.25))
-    (pad "MP" smd roundrect (at -2.475 1.35 180) (size 1 2.7) (layers "F.Cu" "F.Paste" "F.Mask") (roundrect_rratio 0.25))
+    (pad "MP" smd roundrect (at 2.475 1.35 180) (size 1 2.7) (layers "F.Cu" "F.Paste" "F.Mask") (roundrect_rratio 0.25)
+      (net 1 "GND"))
+    (pad "MP" smd roundrect (at -2.475 1.35 180) (size 1 2.7) (layers "F.Cu" "F.Paste" "F.Mask") (roundrect_rratio 0.25)
+      (net 1 "GND"))
     (model "${KICAD6_3DMODEL_DIR}/Connector_JST.3dshapes/JST_GH_SM02B-GHS-TB_1x02-1MP_P1.25mm_Horizontal.wrl"
       (offset (xyz 0 0 0))
@@
     (property "Sheetname" "")
     (attr smd)
-    (fp_text reference "D4" (at -2.8 1.55 90 unlocked) (layer "F.SilkS")
-      (effects (font (size 1 1) (thickness 0.15)))
-    )
+    (fp_text reference "D3" (at -2.8 1.55 90 unlocked) (layer "F.SilkS")
+      (effects (font (size 1 1) (thickness 0.15)))
+    )

Commit message: Use more appropriate J2 symbol to prevent DRC warning
Parts:
- J2: value Conn_01x02 -> Conn_01x02_MountingPin
Changed lines of the file:
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@@
       (effects (font (size 1 1) (thickness 0.15)))
     )
-    (fp_text value "Conn_01x02" (at 0 3.9) (layer "F.Fab")
+    (fp_text value "Conn_01x02_MountingPin" (at 0 3.9) (layer "F.Fab")
       (effects (font (size 1 1) (thickness 0.15)))
     )
@@
       (net 1 "GND") (pinfunction "Pin_2") (pintype "passive"))
     (pad "MP" smd roundrect (at 2.475 1.35 180) (size 1 2.7) (layers "F.Cu" "F.Paste" "F.Mask") (roundrect_rratio 0.25)
-      (net 1 "GND"))
+      (net 1 "GND") (pinfunction "MountPin") (pintype "passive"))
     (pad "MP" smd roundrect (at -2.475 1.35 180) (size 1 2.7) (layers "F.Cu" "F.Paste" "F.Mask") (roundrect_rratio 0.25)
-      (net 1 "GND"))
+      (net 1 "GND") (pinfunction "MountPin") (pintype "passive"))
     (model "${KICAD6_3DMODEL_DIR}/Connector_JST.3dshapes/JST_GH_SM02B-GHS-TB_1x02-1MP_P1.25mm_Horizontal.wrl"
       (offset (xyz 0 0 0))
